File: LM317 PSU.sch (EAGLE design)
At the start: 23 parts, among them IC1 7815

Commit message: Updated Eagle files after mistake noticed
Parts:
- removed R4: 1R - 5W, adafruit:R-US_V234/12
Connections:
- removed net N$9: R4.1
- net N$15: no longer R4.2
Changed lines of the file:
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@@
 <part name="IC1" library="SparkFun" deviceset="V_REG_78XX" device="SINK" value="7815"/>
 <part name="R1" library="adafruit" deviceset="R-US_" device="V234/12" value="1k - 5W"/>
-<part name="R4" library="adafruit" deviceset="R-US_" device="V234/12" value="1R - 5W"/>
 </parts>
 <sheets>
@@
 <instance part="IC1" gate="G$1" x="147.32" y="134.62"/>
 <instance part="R1" gate="G$1" x="96.52" y="76.2" rot="R90"/>
-<instance part="R4" gate="G$1" x="205.74" y="114.3" smashed="yes" rot="R90">
-<attribute name="NAME" x="204.2414" y="110.49" size="1.778" layer="95" rot="R90"/>
-<attribute name="VALUE" x="203.962" y="115.57" size="1.778" layer="96" rot="R90"/>
-</instance>
 </instances>
 <busses>
@@
 <pinref part="JP3" gate="G$1" pin="2"/>
 <wire x1="208.28" y1="88.9" x2="208.28" y2="96.52" width="0.1524" layer="91"/>
-<pinref part="R4" gate="G$1" pin="2"/>
-<wire x1="205.74" y1="119.38" x2="205.74" y2="121.92" width="0.1524" layer="91"/>
-<wire x1="205.74" y1="121.92" x2="208.28" y2="121.92" width="0.1524" layer="91"/>
-<wire x1="208.28" y1="121.92" x2="208.28" y2="96.52" width="0.1524" layer="91"/>
 </segment>
 </net>
@@
 </segment>
 </net>
-<net name="N$9" class="0">
-<segment>
-<pinref part="R4" gate="G$1" pin="1"/>
-<wire x1="205.74" y1="101.6" x2="205.74" y2="109.22" width="0.1524" layer="91"/>
-</segment>
-</net>
